Commit message: changed to 8dof sassa

File: urdf/dog.urdf.xacro (robot description, xacro)
@@ -3,74 +3,56 @@
 dog.urdf.xacro
 ==============
-URDF for the Dog quadruped robot (MIT mini Cheetah-style).
-Physical dimensions (from robot_config.py):
-  Body:        430 mm (L) x 150 mm (W) x 100 mm (H)
-  Hip offset:  130 mm  (abduction link)
-  Upper leg:   320 mm  (femur / shoulder-to-knee)
-  Lower leg:   320 mm  (tibia / knee-to-foot)
-Joint order matches /joint_angles Float32MultiArray:
-  [FR_hip, FR_sho, FR_kne,
-   FL_hip, FL_sho, FL_kne,
-   RR_hip, RR_sho, RR_kne,
-   RL_hip, RL_sho, RL_kne]
-Coordinate convention (ROS standard):
-  x = forward,  y = left,  z = up
+Phase 1 migration base for robotic_dog_clone using the 8-DOF CAD morphology
+from robotic_dog_8dof_urdf, while preserving the clone-side ROS 2 stack.
+Preserved clone-side contracts:
+  - robot name: dog
+  - base frame: base_link
+  - IMU frame:  imu_link
+  - LiDAR frame: lidar_link
+  - shoulder/knee joint names used by gait_node and sim_bridge_node
+  - Gazebo sensor plugins
+  - ros2_control embedding
+Intentional Phase 1 choices:
+  - No base_footprint frame adopted
+  - No hip joints in the active morphology
+  - LiDAR kept level (rpy = 0 0 0) to preserve planar scan assumption
 -->
 <robot name="dog" xmlns:xacro="http://www.ros.org/wiki/xacro">
-  <!-- ═══════════════════════════════════════════════════════════════
-       Parameters
-  ═══════════════════════════════════════════════════════════════ -->
-  <xacro:property name="body_l"     value="0.430"/>
-  <xacro:property name="body_w"     value="0.150"/>
-  <xacro:property name="body_h"     value="0.100"/>
-  <xacro:property name="body_mass"  value="4.0"/>
-  <xacro:property name="hip_offset" value="0.130"/>
-  <xacro:property name="upper_len"  value="0.320"/>
-  <xacro:property name="lower_len"  value="0.320"/>
-  <xacro:property name="foot_r"     value="0.030"/>
-  <xacro:property name="hip_mass"   value="0.300"/>
-  <xacro:property name="upper_mass" value="0.500"/>
-  <xacro:property name="lower_mass" value="0.300"/>
-  <xacro:property name="foot_mass"  value="0.050"/>
-  <!-- Mesh scale factors: mini-Cheetah meshes scaled to this robot's dimensions.
-       body : 1.56×0.76×1.01  (mesh 276×197×99 mm → hip spacing 430×150×100 mm)
-       abad : 2.10 uniform     (abad arm 62 mm → 130 mm)
-       upper: 1.53 uniform     (thigh 209 mm → 320 mm)
-       lower: 1.78 uniform     (shank 180 mm → 320 mm)
-       Adjust these if the meshes look off in RViz. -->
-  <xacro:property name="body_ms"  value="1.56 0.76 1.01"/>
-  <xacro:property name="abad_ms"  value="2.10 2.10 2.10"/>
-  <xacro:property name="upper_ms" value="1.53 1.53 1.53"/>
-  <xacro:property name="lower_ms" value="1.78 1.78 1.78"/>
-  <!-- ═══════════════════════════════════════════════════════════════
+  <!-- ──────────────────────────────────────────────────────────────
        Materials
-  ═══════════════════════════════════════════════════════════════ -->
-  <material name="dark_grey">  <color rgba="0.20 0.20 0.20 1.0"/> </material>
-  <material name="light_grey"> <color rgba="0.70 0.70 0.70 1.0"/> </material>
-  <material name="orange">     <color rgba="1.00 0.50 0.00 1.0"/> </material>
-  <!-- ═══════════════════════════════════════════════════════════════
-       Base (torso)
-  ═══════════════════════════════════════════════════════════════ -->
+  ────────────────────────────────────────────────────────────── -->
+  <material name="dark_grey">
+    <color rgba="0.20 0.20 0.20 1.0"/>
+  </material>
+  <!-- ──────────────────────────────────────────────────────────────
+       Base link — migrated from robotic_dog_8dof_urdf/base_link
+       Name preserved as base_link for clone stack compatibility.
+  ────────────────────────────────────────────────────────────── -->
   <link name="base_link">
     <inertial>
-      <origin xyz="0 0 0" rpy="0 0 0"/>
-      <mass value="${body_mass}"/>
-      <!-- ixx=(m/12)*(w²+h²), iyy=(m/12)*(l²+h²), izz=(m/12)*(l²+w²) -->
-      <inertia ixx="0.0108" ixy="0" ixz="0"
-               iyy="0.0650" iyz="0"
-               izz="0.0691"/>
+      <origin xyz="0.0324578171199918 -0.00107208054772986 -0.0532934197949659" rpy="0 0 0"/>
+      <mass value="9.55580178099991"/>
+      <inertia
+        ixx="0.028878887728372"
+        ixy="-5.32734038649637E-05"
+        ixz="-9.99548284777576E-05"
+        iyy="0.0328205453767607"
+        iyz="-2.0005331957631E-05"
+        izz="0.0484423164334583"/>
     </inertial>
     <visual>
       <origin xyz="0 0 0" rpy="0 0 0"/>
       <geometry>
-        <mesh filename="file://$(find dog)/urdf/meshes/body.dae" scale="${body_ms}"/>
+        <mesh filename="file://$(find dog)/urdf/meshes/base_link.STL"/>
       </geometry>
     </visual>
     <collision>
       <origin xyz="0 0 0" rpy="0 0 0"/>
-      <geometry><box size="${body_l} ${body_w} ${body_h}"/></geometry>
+      <geometry>
+        <mesh filename="file://$(find dog)/urdf/meshes/base_link_collisional.STL"/>
+      </geometry>
     </collision>
   </link>
-  <!-- IMU frame -->
+  <!-- IMU frame preserved for clone-side IMU topics / TF -->
   <link name="imu_link"/>
   <joint name="imu_joint" type="fixed">
@@ -79,40 +61,44 @@
     <origin xyz="0 0 0" rpy="0 0 0"/>
   </joint>
-  <!-- ═══════════════════════════════════════════════════════════════
-       Hokuyo UTM-30LX 2-D LiDAR (visual only)
-       Front-mounted, tilted 45° nose-down.  60 × 60 × 87 mm box.
-  ═══════════════════════════════════════════════════════════════ -->
+  <!-- LiDAR frame preserved for clone-side SLAM/Nav2 assumptions.
+       CAD translation kept; pitch intentionally flattened to zero. -->
   <link name="lidar_link">
     <inertial>
       <origin xyz="0 0 0" rpy="0 0 0"/>
       <mass value="0.370"/>
-      <inertia ixx="3.4e-4" ixy="0" ixz="0"
-               iyy="3.4e-4" iyz="0"
-               izz="2.2e-4"/>
+      <inertia
+        ixx="3.4e-4" ixy="0" ixz="0"
+        iyy="3.4e-4" iyz="0"
+        izz="2.2e-4"/>
     </inertial>
     <visual>
       <origin xyz="0 0 0" rpy="0 0 0"/>
-      <geometry><box size="0.060 0.060 0.087"/></geometry>
+      <geometry>
+        <box size="0.060 0.060 0.087"/>
+      </geometry>
       <material name="dark_grey"/>
     </visual>
     <collision>
       <origin xyz="0 0 0" rpy="0 0 0"/>
-      <geometry><box size="0.060 0.060 0.087"/></geometry>
+      <geometry>
+        <box size="0.060 0.060 0.087"/>
+      </geometry>
     </collision>
   </link>
-  <!-- x: clears front face (+0.030 beyond body half-length)
-       z: sits on top of body (+0.044 = half of 87 mm above body top)
-       pitch 0 = horizontal scan plane — required for 2D SLAM.
-       Change rpy to "0 -0.7854 0" if you physically tilt the sensor nose-down. -->
   <joint name="lidar_joint" type="fixed">
     <parent link="base_link"/>
     <child  link="lidar_link"/>
-    <origin xyz="${body_l/2 + 0.030} 0 ${body_h/2 + 0.044}" rpy="0 0 0"/>
+    <origin xyz="0.284282580961245 9.01880488845888E-05 0.0962574459982149" rpy="0 0 0"/>
   </joint>
-  <!-- ═══════════════════════════════════════════════════════════════
-       Gazebo: Hokuyo UTM-30LX lidar sensor (simulation only)
-       Publishes Ignition LaserScan → bridged to /scan by autonomous_launch.
-       270° FOV (-135° to +135°), 720 samples, 30 m max range.
-  ═══════════════════════════════════════════════════════════════ -->
+  <!-- Camera frame imported from CAD model for future use -->
+  <link name="camera_link"/>
+  <joint name="camera_joint" type="fixed">
+    <parent link="base_link"/>
+    <child  link="camera_link"/>
+    <origin xyz="0.352482816608291 0.000734336789502524 -0.0246227904334168" rpy="0 0 0"/>
+  </joint>
+  <!-- ──────────────────────────────────────────────────────────────
+       Gazebo: Hokuyo-style lidar sensor (simulation only)
+  ────────────────────────────────────────────────────────────── -->
   <gazebo reference="lidar_link">
     <sensor name="hokuyo_lidar" type="lidar">
@@ -143,234 +129,240 @@
     </sensor>
   </gazebo>
-  <!-- ═══════════════════════════════════════════════════════════════
-       Leg macro  (kinematics + links only, no ros2_control here)
-       name       : fr | fl | rr | rl
-       bx, by     : body-frame position of hip joint
-       hip_dir    : +1 for left legs (+y), -1 for right legs (-y)
-       sk_axis    : shoulder/knee joint axis.
-                    All legs use "0 1 0": positive angle = upper leg swings backward,
-                    negative knee angle = lower leg bends forward (inward knee).
-                    Matches NEUTRAL_ANGLES sign convention directly.
-       abad_rpy   : rotation to orient the abad mesh correctly for this leg
-       abad_vx_s  : signed x-offset of abad mesh origin (front legs −, rear legs +)
-  ═══════════════════════════════════════════════════════════════ -->
-  <xacro:macro name="leg" params="name bx by hip_dir sk_axis abad_rpy abad_vx_s">
-    <!-- Hip joint: abduction/adduction, axis = +x -->
-    <joint name="${name}_hip_joint" type="revolute">
+  <!-- ──────────────────────────────────────────────────────────────
+       8-DOF leg macro
+       Clone semantic names preserved:
+         fr, fl, rr, rl
+       CAD morphology imported:
+         - one shoulder joint from base_link to upper link
+         - one knee joint from upper link to lower link
+         - axis = 0 1 0 for all active joints
+  ────────────────────────────────────────────────────────────── -->
+  <xacro:macro name="cad_leg" params="
+      name
+      shoulder_xyz
+      knee_xyz
+      upper_mesh
+      upper_collision_mesh
+      upper_com_xyz
+      upper_mass
+      upper_ixx upper_ixy upper_ixz upper_iyy upper_iyz upper_izz
+      lower_mesh
+      lower_collision_mesh
+      lower_com_xyz
+      lower_mass
+      lower_ixx lower_ixy lower_ixz lower_iyy lower_iyz lower_izz">
+    <joint name="${name}_shoulder_joint" type="revolute">
       <parent link="base_link"/>
-      <child  link="${name}_hip_link"/>
-      <origin xyz="${bx} ${by} 0" rpy="0 0 0"/>
-      <axis xyz="1 0 0"/>
-      <limit lower="-0.785" upper="0.785" effort="18.0" velocity="45.0"/>
+      <child  link="${name}_upper_leg_link"/>
+      <origin xyz="${shoulder_xyz}" rpy="0 0 0"/>
+      <axis xyz="0 1 0"/>
+      <limit lower="-2.094" upper="2.094" effort="8" velocity="4.19"/>
       <dynamics damping="0.1" friction="0.0"/>
     </joint>
-    <link name="${name}_hip_link">
+    <link name="${name}_upper_leg_link">
       <inertial>
-        <origin xyz="0 ${hip_dir * hip_offset * 0.5} 0" rpy="0 0 0"/>
-        <mass value="${hip_mass}"/>
-        <!-- cylinder along y: ixx=izz=(m/12)*(3r²+l²), iyy=(m/2)*r² -->
-        <inertia ixx="4.7e-4" ixy="0" ixz="0"
-                 iyy="9.4e-5" iyz="0"
-                 izz="4.7e-4"/>
+        <origin xyz="${upper_com_xyz}" rpy="0 0 0"/>
+        <mass value="${upper_mass}"/>
+        <inertia
+          ixx="${upper_ixx}" ixy="${upper_ixy}" ixz="${upper_ixz}"
+          iyy="${upper_iyy}" iyz="${upper_iyz}"
+          izz="${upper_izz}"/>
       </inertial>
       <visual>
-        <origin xyz="${abad_vx_s} 0 0" rpy="${abad_rpy}"/>
+        <origin xyz="0 0 0" rpy="0 0 0"/>
         <geometry>
-          <mesh filename="file://$(find dog)/urdf/meshes/abad.dae" scale="${abad_ms}"/>
+          <mesh filename="file://$(find dog)/urdf/meshes/${upper_mesh}"/>
         </geometry>
       </visual>
       <collision>
-        <origin xyz="0 ${hip_dir * hip_offset * 0.5} 0" rpy="${pi/2} 0 0"/>
-        <geometry><cylinder radius="0.025" length="${hip_offset}"/></geometry>
+        <origin xyz="0 0 0" rpy="0 0 0"/>
+        <geometry>
+          <mesh filename="file://$(find dog)/urdf/meshes/${upper_collision_mesh}"/>
+        </geometry>
       </collision>
     </link>
-    <!-- Shoulder joint: thigh flexion -->
-    <joint name="${name}_shoulder_joint" type="revolute">
-      <parent link="${name}_hip_link"/>
-      <child  link="${name}_upper_leg_link"/>
-      <origin xyz="0 ${hip_dir * hip_offset} 0" rpy="0 0 0"/>
-      <axis xyz="${sk_axis}"/>
-      <limit lower="-2.618" upper="2.618" effort="50.0" velocity="45.0"/>
+    <joint name="${name}_knee_joint" type="revolute">
+      <parent link="${name}_upper_leg_link"/>
+      <child  link="${name}_lower_leg_link"/>
+      <origin xyz="${knee_xyz}" rpy="0 0 0"/>
+      <axis xyz="0 1 0"/>
+      <limit lower="-2.4" upper="2.4" effort="8" velocity="4.19"/>
       <dynamics damping="0.1" friction="0.0"/>
     </joint>
-    <link name="${name}_upper_leg_link">
+    <link name="${name}_lower_leg_link">
       <inertial>
-        <origin xyz="0 0 ${-upper_len * 0.5}" rpy="0 0 0"/>
-        <mass value="${upper_mass}"/>
-        <!-- cylinder along z: ixx=iyy=(m/12)*(3r²+l²), izz=(m/2)*r² -->
-        <inertia ixx="4.34e-3" ixy="0" ixz="0"
-                 iyy="4.34e-3" iyz="0"
-                 izz="1.56e-4"/>
+        <origin xyz="${lower_com_xyz}" rpy="0 0 0"/>
+        <mass value="${lower_mass}"/>
+        <inertia
+          ixx="${lower_ixx}" ixy="${lower_ixy}" ixz="${lower_ixz}"
+          iyy="${lower_iyy}" iyz="${lower_iyz}"
+          izz="${lower_izz}"/>
       </inertial>
       <visual>
-        <origin xyz="0 0 0" rpy="0 -1.5708 0"/>
+        <origin xyz="0 0 0" rpy="0 0 0"/>
         <geometry>
-          <mesh filename="file://$(find dog)/urdf/meshes/upper_link.dae" scale="${upper_ms}"/>
+          <mesh filename="file://$(find dog)/urdf/meshes/${lower_mesh}"/>
         </geometry>
       </visual>
       <collision>
-        <origin xyz="0 0 ${-upper_len * 0.5}" rpy="0 0 0"/>
-        <geometry><cylinder radius="0.025" length="${upper_len}"/></geometry>
+        <origin xyz="0 0 0" rpy="0 0 0"/>
+        <geometry>
+          <mesh filename="file://$(find dog)/urdf/meshes/${lower_collision_mesh}"/>
+        </geometry>
       </collision>
     </link>
-    <!-- Knee joint: shank flexion -->
-    <joint name="${name}_knee_joint" type="revolute">
-      <parent link="${name}_upper_leg_link"/>
-      <child  link="${name}_lower_leg_link"/>
-      <origin xyz="0 0 ${-upper_len}" rpy="0 0 0"/>
-      <axis xyz="${sk_axis}"/>
-      <limit lower="-2.618" effort="50.0" upper="2.618" velocity="45.0"/>
-      <dynamics damping="0.1" friction="0.0"/>
-    </joint>
-    <link name="${name}_lower_leg_link">
-      <inertial>
-        <origin xyz="0 0 ${-lower_len * 0.5}" rpy="0 0 0"/>
-        <mass value="${lower_mass}"/>
-        <!-- cylinder along z: ixx=iyy=(m/12)*(3r²+l²), izz=(m/2)*r² -->
-        <inertia ixx="2.58e-3" ixy="0" ixz="0"
-                 iyy="2.58e-3" iyz="0"
-                 izz="3.4e-5"/>
-      </inertial>
-      <visual>
-        <origin xyz="0 0 0" rpy="0 3.141592 0"/>
-        <geometry>
-          <mesh filename="file://$(find dog)/urdf/meshes/lower_link.dae" scale="${lower_ms}"/>
-        </geometry>
-      </visual>
-      <collision>
-        <origin xyz="0 0 ${-lower_len * 0.5}" rpy="0 0 0"/>
-        <geometry><cylinder radius="0.018" length="${lower_len}"/></geometry>
-      </collision>
-    </link>
-    <!-- Foot sphere (contact) -->
-    <joint name="${name}_foot_joint" type="fixed">
-      <parent link="${name}_lower_leg_link"/>
-      <child  link="${name}_foot_link"/>
-      <origin xyz="0 0 ${-lower_len}" rpy="0 0 0"/>
-    </joint>
-    <link name="${name}_foot_link">
-      <inertial>
-        <mass value="${foot_mass}"/>
-        <!-- sphere: ixx=iyy=izz=(2/5)*m*r² -->
-        <inertia ixx="1.8e-5" ixy="0" ixz="0"
-                 iyy="1.8e-5" iyz="0"
-                 izz="1.8e-5"/>
-      </inertial>
-      <visual>
-        <geometry><sphere radius="${foot_r}"/></geometry>
-        <material name="orange"/>
-      </visual>
-      <collision>
-        <geometry><sphere radius="${foot_r}"/></geometry>
-      </collision>
-    </link>
-    <!-- Gazebo contact / friction params for this foot -->
-    <gazebo reference="${name}_foot_link">
-      <mu1>1.2</mu1>
-      <mu2>1.2</mu2>
-      <kp>500000.0</kp>
-      <kd>10.0</kd>
-      <minDepth>0.001</minDepth>
-    </gazebo>
   </xacro:macro>
-  <!-- ═══════════════════════════════════════════════════════════════
-       Instantiate legs
-       Neutral standing angles (robot_config.py NEUTRAL_ANGLES):
-         All legs: hip=±0.27, shoulder=+0.57, knee=-1.13 (geometric)
-         controller knee cmd = -0.57 (belt-coupled motor value)
-       (UPPER=320 mm, LOWER=320 mm, STAND_HEIGHT=540 mm)
-  ═══════════════════════════════════════════════════════════════ -->
-  <!-- Inward-facing knees (MIT mini Cheetah style):
-       All legs use "0 1 0": positive shoulder = upper leg backward,
-       negative knee = lower leg forward → knee protrudes inward/backward.
-       This matches the sign convention in NEUTRAL_ANGLES for all four legs.
-       abad_rpy / abad_vx_s orient the abad mesh correctly per leg (from mini_cheetah URDF). -->
-  <xacro:leg name="fr" bx=" 0.215" by="-0.075" hip_dir="-1" sk_axis="0 1 0"
-             abad_rpy="3.141592 0 1.5708"  abad_vx_s="-0.115"/>
-  <xacro:leg name="fl" bx=" 0.215" by=" 0.075" hip_dir=" 1" sk_axis="0 1 0"
-             abad_rpy="0 0 -1.5708"        abad_vx_s="-0.115"/>
-  <xacro:leg name="rr" bx="-0.215" by="-0.075" hip_dir="-1" sk_axis="0 1 0"
-             abad_rpy="0 0 1.5708"         abad_vx_s=" 0.115"/>
-  <xacro:leg name="rl" bx="-0.215" by=" 0.075" hip_dir=" 1" sk_axis="0 1 0"
-             abad_rpy="3.141592 0 -1.5708" abad_vx_s=" 0.115"/>
-  <!-- ═══════════════════════════════════════════════════════════════
-       ros2_control hardware interface (ign_ros2_control)
-       Joint order MUST match /joint_angles Float32MultiArray index:
-         0  fr_hip    3  fl_hip    6  rr_hip    9  rl_hip
-         1  fr_sho    4  fl_sho    7  rr_sho   10  rl_sho
-         2  fr_kne    5  fl_kne    8  rr_kne   11  rl_kne
-  ═══════════════════════════════════════════════════════════════ -->
+  <!-- Front Right = CAD leg2 -->
+  <xacro:cad_leg
+    name="fr"
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
Commit message: earthgjk

File: urdf/dog.urdf.xacro (robot description, xacro)
@@ -1,31 +1,24 @@
 <?xml version="1.0"?>
-<!--
-dog.urdf.xacro
-==============
-Phase 1 migration base for robotic_dog_clone using the 8-DOF CAD morphology
-from robotic_dog_8dof_urdf, while preserving the clone-side ROS 2 stack.
-Preserved clone-side contracts:
-  - robot name: dog
-  - base frame: base_link
-  - IMU frame:  imu_link
-  - LiDAR frame: lidar_link
-  - shoulder/knee joint names used by gait_node and sim_bridge_node
-  - Gazebo sensor plugins
-  - ros2_control embedding
-Intentional Phase 1 choices:
-  - No base_footprint frame adopted
-  - No hip joints in the active morphology
-  - LiDAR kept level (rpy = 0 0 0) to preserve planar scan assumption
--->
 <robot name="dog" xmlns:xacro="http://www.ros.org/wiki/xacro">
   <!-- ──────────────────────────────────────────────────────────────
-       Materials
+       Materials — Virginia Tech brand colors
+         Chicago Maroon  #861F41  → upper legs
+         Burnt Orange    #E5751F  → lower legs
+         Hokie Stone     #75787B  → base / body
   ────────────────────────────────────────────────────────────── -->
   <material name="dark_grey">
     <color rgba="0.20 0.20 0.20 1.0"/>
   </material>
+  <material name="hokie_stone">
+    <color rgba="0.459 0.471 0.482 1.0"/>
+  </material>
+  <material name="chicago_maroon">
+    <color rgba="0.525 0.122 0.255 1.0"/>
+  </material>
+  <material name="burnt_orange">
+    <color rgba="0.898 0.459 0.122 1.0"/>
+  </material>
   <!-- ──────────────────────────────────────────────────────────────
-       Base link — migrated from robotic_dog_8dof_urdf/base_link
-       Name preserved as base_link for clone stack compatibility.
+       Base link
   ────────────────────────────────────────────────────────────── -->
   <link name="base_link">
@@ -46,4 +39,5 @@
         <mesh filename="file://$(find dog)/urdf/meshes/base_link.STL"/>
       </geometry>
+      <material name="hokie_stone"/>
     </visual>
     <collision>
@@ -54,6 +48,14 @@
     </collision>
   </link>
-  <!-- IMU frame preserved for clone-side IMU topics / TF -->
-  <link name="imu_link"/>
+  <!-- IMU frame -->
+  <link name="imu_link">
+    <inertial>
+      <mass value="0.001"/>
+      <origin xyz="0 0 0" rpy="0 0 0"/>
+      <inertia ixx="1e-6" ixy="0" ixz="0"
+              iyy="1e-6" iyz="0"
+              izz="1e-6"/>
+    </inertial>
+  </link>
   <joint name="imu_joint" type="fixed">
     <parent link="base_link"/>
@@ -61,6 +63,5 @@
     <origin xyz="0 0 0" rpy="0 0 0"/>
   </joint>
-  <!-- LiDAR frame preserved for clone-side SLAM/Nav2 assumptions.
-       CAD translation kept; pitch intentionally flattened to zero. -->
+  <!-- LiDAR frame -->
   <link name="lidar_link">
     <inertial>
@@ -91,5 +92,5 @@
     <origin xyz="0.284282580961245 9.01880488845888E-05 0.0962574459982149" rpy="0 0 0"/>
   </joint>
-  <!-- Camera frame imported from CAD model for future use -->
+  <!-- Camera frame -->
   <link name="camera_link"/>
   <joint name="camera_joint" type="fixed">
@@ -99,5 +100,5 @@
   </joint>
   <!-- ──────────────────────────────────────────────────────────────
-       Gazebo: Hokuyo-style lidar sensor (simulation only)
+       Gazebo: Hokuyo-style lidar sensor
   ────────────────────────────────────────────────────────────── -->
   <gazebo reference="lidar_link">
@@ -131,10 +132,6 @@
   <!-- ──────────────────────────────────────────────────────────────
        8-DOF leg macro
-       Clone semantic names preserved:
-         fr, fl, rr, rl
-       CAD morphology imported:
-         - one shoulder joint from base_link to upper link
-         - one knee joint from upper link to lower link
-         - axis = 0 1 0 for all active joints
+       Upper leg → Chicago Maroon
+       Lower leg → Burnt Orange
   ────────────────────────────────────────────────────────────── -->
   <xacro:macro name="cad_leg" params="
@@ -174,4 +171,5 @@
           <mesh filename="file://$(find dog)/urdf/meshes/${upper_mesh}"/>
         </geometry>
+        <material name="chicago_maroon"/>
       </visual>
       <collision>
@@ -204,4 +202,5 @@
           <mesh filename="file://$(find dog)/urdf/meshes/${lower_mesh}"/>
         </geometry>
+        <material name="burnt_orange"/>
       </visual>
       <collision>
@@ -314,9 +313,5 @@
     lower_izz="1.77307368033845E-05"/>
   <!-- ──────────────────────────────────────────────────────────────
-       ros2_control hardware interface (kept in-file for clone stack)
-       Active joints only: 8DOF shoulder + knee
-       Initial values chosen to match current clone neutral motor model:
-         shoulder ≈ +0.6112
-         geometric knee ≈ -1.2224
+       ros2_control hardware interface
   ────────────────────────────────────────────────────────────── -->
   <ros2_control name="GazeboSimSystem" type="system">
@@ -365,5 +360,5 @@
     </joint>
   </ros2_control>
-  <!-- ign_ros2_control: starts controller_manager inside Gazebo -->
+  <!-- ign_ros2_control plugin -->
   <gazebo>
     <plugin filename="ign_ros2_control-system"
